Commit message: fix(tf): align left depth camera frame

File: realbots2/urdf/realbots29.urdf (robot description, URDF)
Before this commit: robot realbots29, 56 links, 55 joints
Joints:
- joint left_binocular_left_camera_joint: origin xyz=0.0490945700197835 0 -0.000100000000000211 rpy=0 0 0 -> xyz=0.0490945700197835 0 -0.000100000000000211 rpy=-0.087266462599716 0 0
- joint left_binocular_right_camera_joint: origin xyz=-0.0459054299802165 0 -0.000100000000000156 rpy=0 0 0 -> xyz=-0.0459054299802165 0 -0.000100000000000156 rpy=-0.087266462599716 0 0
- joint left_rgb_camera_Link: origin xyz=0.0253455085535028 0 -0.000100000000000211 rpy=0 0 0 -> xyz=0.0253455085535028 0 -0.000100000000000211 rpy=-0.087266462599716 0 0
- joint left_speckle_camera_joint: origin xyz=0.00159547181944711 0 -0.000100000000000156 rpy=0 0 0 -> xyz=0.00159547181944711 0 -0.000100000000000156 rpy=-0.087266462599716 0 0
